Commit message: fix axis and dimensions

File: robot_description/urdf/robot_hand.urdf (robot description, URDF)
Before this commit: robot robot_hand, 17 links, 16 joints
Links:
- link thumb_middle: geometry visual cylinder length=0.03 radius=0.008
- link thumb_proximal: geometry visual cylinder length=0.03 radius=0.009
Joints:
- joint index_dip: axis 0 1 0 -> 1 0 0
- joint index_mcp: axis 0 1 0 -> 1 0 0
- joint index_pip: axis 0 1 0 -> 1 0 0
- joint middle_dip: axis 0 1 0 -> 1 0 0
- joint middle_mcp: axis 0 1 0 -> 1 0 0
- joint middle_pip: axis 0 1 0 -> 1 0 0
- joint pinky_dip: axis 0 1 0 -> 1 0 0
- joint pinky_mcp: axis 0 1 0 -> 1 0 0
- joint pinky_pip: axis 0 1 0 -> 1 0 0
- joint ring_dip: axis 0 1 0 -> 1 0 0
- joint ring_mcp: axis 0 1 0 -> 1 0 0
- joint ring_pip: axis 0 1 0 -> 1 0 0
- joint thumb_dip: axis 0 1 0 -> -1 0 0; origin xyz=0 0 0.036 -> xyz=0 0 0.03
- joint thumb_mcp: axis 0 1 0 -> -1 0 0; origin xyz=0.045 -0.025 0.01 rpy=0 0 0.8 -> xyz=0.045 -0.025 0.01 rpy=0 0 1.3
- joint thumb_pip: axis 0 1 0 -> -1 0 0; origin xyz=0 0 0.04 -> xyz=0 0 0.03
